Commit message: Phase 5.1: SLAM mapping and dynamic safety remediation
Root cause: the headless gpu_lidar renderer (Mesa zink-on-NVK) drew
only the forward camera face, so the front LiDAR saw +/-45 deg and the
360 scanner was mostly blind; phantom returns became map streaks.

- sim.launch.py: NOUVEAU_USE_ZINK=0; audit fails on a blind front
  sector; validate_lidar_rendering.py checks beams against geometry
- SLAM: Phase 5 matcher kept; loop search narrowed to 1.5 m / 3 m
  (identical aisles 4.2 m apart caused false closures)
- odometry_wheel_separation 0.5258 m through the generator
- 360 elevated scanner via the pipeline (params, Blender, URDF,
  Gazebo, bridge, GLB), own Nav2 obstacle layer, guard requirement
- HumanSystem worker yielding (forces only, bounded wait)
- mapping_jog refuses unobserved rotations; survey plans, bag
  recording, offline replay, candidate evaluation workflow
- approved full-warehouse map v11 (operator-approved): 6 stations,
  30/30 station pairs, 3 cycles; registration and graph rebuilt
- execute_route deadline in simulation time; registration offsets
  consolidated in coordinate_registration.active()
- docs: PHASE_5_1_REMEDIATION.md, PHASE_5_1_VALIDATION.md,
  Phase 5 addenda and summaries

Co-Authored-By: Claude Opus 5.5 <noreply@anthropic.com>

File: src/amr_description/urdf/amr.urdf.xacro (robot description, xacro)
@@ -14,4 +14,5 @@
   <xacro:include filename="components/casters.xacro"/>
   <xacro:include filename="sensors/lidar.xacro"/>
+  <xacro:include filename="sensors/top_lidar.xacro"/>
   <xacro:include filename="sensors/imu.xacro"/>
   <xacro:include filename="sensors/camera.xacro"/>
@@ -27,5 +28,5 @@
   <link name="base_link"/>
   <xacro:chassis/><xacro:platform/><xacro:wheels/><xacro:casters/>
-  <xacro:lidar/><xacro:imu debug="$(arg debug_imu)"/><xacro:camera/>
+  <xacro:lidar/><xacro:top_lidar/><xacro:imu debug="$(arg debug_imu)"/><xacro:camera/>
   <xacro:if value="$(arg gazebo)">
     <xacro:gazebo_properties/><xacro:gazebo_sensors/>

File: src/amr_description/urdf/dimensions.xacro (robot description, xacro)
@@ -18,4 +18,5 @@
   <xacro:property name="wheel_width" value="0.055"/>
   <xacro:property name="track_width" value="0.58"/>
+  <xacro:property name="odometry_wheel_separation" value="0.5258"/>
   <xacro:property name="wheel_arch_gap" value="0.009"/>
   <xacro:property name="wheel_bevel" value="0.003"/>
@@ -65,4 +66,15 @@
   <xacro:property name="lidar_max_range" value="20"/>
   <xacro:property name="lidar_resolution" value="0.01"/>
+  <xacro:property name="top_lidar_rear_inset" value="0.06"/>
+  <xacro:property name="top_lidar_mast_radius" value="0.018"/>
+  <xacro:property name="top_lidar_clearance" value="0.08"/>
+  <xacro:property name="top_lidar_radius" value="0.04"/>
+  <xacro:property name="top_lidar_height" value="0.05"/>
+  <xacro:property name="top_lidar_mass" value="0.4"/>
+  <xacro:property name="top_lidar_mast_mass" value="0.25"/>
+  <xacro:property name="top_lidar_samples" value="720"/>
+  <xacro:property name="top_lidar_rate" value="10"/>
+  <xacro:property name="top_lidar_min_range" value="0.12"/>
+  <xacro:property name="top_lidar_max_range" value="20"/>
   <xacro:property name="imu_rate" value="100"/>
   <xacro:property name="camera_rate" value="15"/>
@@ -104,4 +116,9 @@
   <xacro:property name="camera_z" value="0.264"/>
   <xacro:property name="lidar_half_fov" value="1.57079632679"/>
+  <xacro:property name="top_lidar_x" value="-0.38"/>
+  <xacro:property name="top_mast_z" value="0.384"/>
+  <xacro:property name="top_lidar_z" value="0.449"/>
+  <xacro:property name="top_laser_z" value="0.48"/>
+  <xacro:property name="top_lidar_angle_step" value="0.00872664625997"/>
   <xacro:property name="camera_fov" value="1.308996939"/>
   <xacro:property name="core_length" value="0.868"/>

File: src/amr_description/urdf/gazebo/sensors_gazebo.xacro (robot description, xacro)
@@ -10,4 +10,15 @@
           <min_angle>${-lidar_half_fov}</min_angle><max_angle>${lidar_half_fov}</max_angle>
         </horizontal></scan><range><min>${lidar_min_range}</min><max>${lidar_max_range}</max><resolution>${lidar_resolution}</resolution></range></lidar>
+      </sensor>
+    </gazebo>
+    <gazebo reference="top_lidar_link">
+      <!-- Full circle without a duplicated beam at +/-pi. -->
+      <sensor name="top_lidar" type="gpu_lidar">
+        <pose>0 0 ${top_laser_z-top_lidar_z} 0 0 0</pose>
+        <topic>/amr/top_scan</topic><gz_frame_id>top_laser_frame</gz_frame_id>
+        <always_on>true</always_on><update_rate>${top_lidar_rate}</update_rate><visualize>false</visualize>
+        <lidar><scan><horizontal><samples>${top_lidar_samples}</samples><resolution>1</resolution>
+          <min_angle>${-pi}</min_angle><max_angle>${pi-top_lidar_angle_step}</max_angle>
+        </horizontal></scan><range><min>${top_lidar_min_range}</min><max>${top_lidar_max_range}</max><resolution>${lidar_resolution}</resolution></range></lidar>
       </sensor>
     </gazebo>
